File: 120-channel-pogo-pin-board.sch (KiCad schematic (older format))
At the start: 17 parts, among them J4 SFM-120-02-L-D-A, J5 SFM-125-02-L-D-A, J6 SFM-120-02-L-D-A, P1 Conn_02x17_Odd_Even, P2 Conn_02x17_Odd_Even, P3 Conn_02x17_Odd_Even, P4 Conn_02x17_Odd_Even, P5 CONN_01X01, P6 CONN_01X01, P7 CONN_01X01, P8 CONN_01X01, U1 CAT24C02TDI

Commit message: Update to kicad 5
Parts:
- C1, C2: symbol C -> Device:C
- R1: symbol R_Small -> Device:R_Small
Connections:
- wire segments 20 -> 28
Changed lines of the file:
@@
-EESchema Schematic File Version 2
-LIBS:120-channel pogo pin board-rescue
-LIBS:power
-LIBS:device
-LIBS:transistors
-LIBS:conn
-LIBS:linear
-LIBS:regul
-LIBS:74xx
-LIBS:cmos4000
-LIBS:adc-dac
-LIBS:memory
-LIBS:xilinx
-LIBS:microcontrollers
-LIBS:dsp
-LIBS:microchip
-LIBS:analog_switches
-LIBS:motorola
-LIBS:texas
-LIBS:intel
-LIBS:audio
-LIBS:interface
-LIBS:digital-audio
-LIBS:philips
-LIBS:display
-LIBS:cypress
-LIBS:siliconi
-LIBS:opto
-LIBS:atmel
-LIBS:contrib
-LIBS:valves
-LIBS:sci-bots
-LIBS:120-channel pogo pin board-cache
-EELAYER 25 0
+EESchema Schematic File Version 4
+EELAYER 30 0
 EELAYER END
 $Descr User 11000 8500
@@
 $EndComp
 Wire Wire Line
-	950  1550 1200 1550
+	950  1550 1050 1550
 Wire Wire Line
 	2400 1550 2300 1550
 Wire Wire Line
-	2400 1350 2400 1550
+	2400 1350 2400 1450
 Connection ~ 1050 1550
 Wire Wire Line
-	2300 1450 2550 1450
+	2300 1450 2400 1450
 Connection ~ 2400 1450
 Wire Wire Line
@@
 Connection ~ 1050 1450
 $Comp
-L C C1
+L Device:C C1
 U 1 1 58C0BBB2
 P 950 1100
@@
 GND
 Wire Wire Line
-	950  900  1450 900
+	950  900  1150 900
 Wire Wire Line
 	950  900  950  950
@@
 	1150 1350 1150 1250
 Wire Wire Line
-	950  1350 1150 1350
+	950  1350 1050 1350
 Wire Wire Line
 	950  1350 950  1250
@@
 CHASIS_GND
 $Comp
-L C C2
+L Device:C C2
 U 1 1 58C0D9E0
 P 2300 1100
@@
 GND
 Wire Wire Line
-	2300 900  2800 900
+	2300 900  2500 900
 Wire Wire Line
 	2300 900  2300 950
@@
 	2500 1350 2500 1250
 Wire Wire Line
-	2300 1350 2500 1350
+	2300 1350 2400 1350
 Wire Wire Line
 	2300 1350 2300 1250
 Connection ~ 2400 1350
 Wire Wire Line
-	1050 1350 1050 1550
+	1050 1350 1050 1450
 $Comp
 L CAT24C__TD_ U1
@@
 GND
 $Comp
-L R_Small R1
+L Device:R_Small R1
 U 1 1 58C170A6
 P 6050 3800
@@
 	-1   0    0    1
 $EndComp
+Wire Wire Line
+	1050 1550 1200 1550
+Wire Wire Line
+	2400 1450 2400 1550
+Wire Wire Line
+	2400 1450 2550 1450
+Wire Wire Line
+	1050 1450 1050 1550
+Wire Wire Line
+	1150 900  1450 900
+Wire Wire Line
+	1050 1350 1150 1350
+Wire Wire Line
+	2500 900  2800 900
+Wire Wire Line
+	2400 1350 2500 1350
 $EndSCHEMATC

Commit message: Fix broken symbols
Parts:
- FB1, FB2: symbol FERRITE -> Device:Ferrite_Bead_Small
- J4, J6: symbol CONN_02X20 -> Connector_Generic:Conn_02x20_Odd_Even
- J5: symbol CONN_02X25 -> Connector_Generic:Conn_02x25_Odd_Even
- P1, P2, P3, P4: symbol CONN_02X17 -> Connector_Generic:Conn_02x17_Odd_Even
- P5, P6, P7, P8: symbol CONN_01X01 -> Connector_Generic:Conn_01x01
- U1: symbol CAT24C__TD_ -> sci-bots:CAT24C__TD_
Changed lines of the file:
@@
 CHASIS_GND
 $Comp
-L CONN_01X01 P5
+L Connector_Generic:Conn_01x01 P5
 U 1 1 58C0AD0D
 P 750 1550
@@
 $EndComp
 $Comp
-L CONN_01X01 P6
+L Connector_Generic:Conn_01x01 P6
 U 1 1 58C0AD4A
 P 2100 1450
@@
 $EndComp
 $Comp
-L CONN_01X01 P7
+L Connector_Generic:Conn_01x01 P7
 U 1 1 58C0AD75
 P 750 1450
@@
 $EndComp
 $Comp
-L CONN_01X01 P8
+L Connector_Generic:Conn_01x01 P8
 U 1 1 58C0ADA3
 P 2100 1550
@@
 $EndComp
 $Comp
-L FERRITE FB1
+L Device:Ferrite_Bead_Small FB1
 U 1 1 58C0D2EB
-P 1150 1100
-F 0 "FB1" H 1025 1275 50  0000 L CNN
-F 1 "FERRITE" H 1025 1200 50  0000 L CNN
-F 2 "Resistors_SMD:R_0805" H 1150 1000 60  0001 C CNN
-F 3 "" H 1150 1000 60  0000 C CNN
-F 4 "742792040" H 1150 1100 60  0001 C CNN "Mfg_Part_No"
-	1    1150 1100
-	0    1    1    0
+P 1150 1050
+F 0 "FB1" H 900 1150 50  0000 L CNN
+F 1 "FERRITE" H 750 1050 50  0000 L CNN
+F 2 "Resistors_SMD:R_0805" H 1150 950 60  0001 C CNN
+F 3 "" H 1150 950 60  0000 C CNN
+F 4 "742792040" H 1150 1050 60  0001 C CNN "Mfg_Part_No"
+	1    1150 1050
+	-1   0    0    1
 $EndComp
 Text GLabel 1450 900  2    60   Input ~ 0
@@
 	1150 950  1150 900
 Connection ~ 1150 900
-Wire Wire Line
-	1150 1350 1150 1250
 Wire Wire Line
 	950  1350 1050 1350
@@
 $EndComp
 $Comp
-L FERRITE FB2
+L Device:Ferrite_Bead_Small FB2
 U 1 1 58C0D9E6
-P 2500 1100
-F 0 "FB2" H 2375 1275 50  0000 L CNN
-F 1 "FERRITE" H 2375 1200 50  0000 L CNN
-F 2 "Resistors_SMD:R_0805" H 2500 1000 60  0001 C CNN
-F 3 "" H 2500 1000 60  0000 C CNN
-F 4 "742792040" H 2500 1100 60  0001 C CNN "Mfg_Part_No"
-	1    2500 1100
-	0    1    1    0
+P 2500 1050
+F 0 "FB2" H 2250 1150 50  0000 L CNN
+F 1 "FERRITE" H 2100 1050 50  0000 L CNN
+F 2 "Resistors_SMD:R_0805" H 2500 950 60  0001 C CNN
+F 3 "" H 2500 950 60  0000 C CNN
+F 4 "742792040" H 2500 1050 60  0001 C CNN "Mfg_Part_No"
+	1    2500 1050
+	-1   0    0    1
 $EndComp
 Text GLabel 2800 900  2    60   Input ~ 0
@@
 Connection ~ 2500 900
 Wire Wire Line
-	2500 1350 2500 1250
-Wire Wire Line
 	2300 1350 2400 1350
 Wire Wire Line
@@
 	1050 1350 1050 1450
 $Comp
-L CAT24C__TD_ U1
+L sci-bots:CAT24C__TD_ U1
 U 1 1 58C15955
 P 5650 3950
@@
 P 6050 3800
 F 0 "R1" V 6150 3750 50  0000 L CNN
-F 1 "10k" V 6050 3750 50  0000 L CNN
+F 1 "10k" V 5950 3750 50  0000 L CNN
 F 2 "Resistors_SMD:R_0805" H 6050 3800 50  0001 C CNN
 F 3 "" H 6050 3800 50  0000 C CNN
@@
 EEPROM 2k
 $Comp
-L CONN_02X17 P2
+L Connector_Generic:Conn_02x17_Odd_Even P2
 U 1 1 5A4F0D39
-P 1300 5500
-F 0 "P2" H 1350 6400 50  0000 C CNN
-F 1 "Conn_02x17_Odd_Even" H 1350 4600 50  0000 C CNN
-F 2 "Sci-Bots:Pogo_Pin_Header_Straight_2x17_Pitch2.54mm" H 1300 5500 50  0001 C CNN
-F 3 "" H 1300 5500 50  0001 C CNN
-F 4 "823-22-034-10-000101" H 1300 5500 60  0001 C CNN "Mfg_Part_No"
-	1    1300 5500
-	1    0    0    -1
-$EndComp
-$Comp
-L CONN_02X17 P1
+P 1250 5500
+F 0 "P2" H 1300 6400 50  0000 C CNN
+F 1 "Conn_02x17_Odd_Even" H 1300 4600 50  0000 C CNN
+F 2 "Sci-Bots:Pogo_Pin_Header_Straight_2x17_Pitch2.54mm" H 1250 5500 50  0001 C CNN
+F 3 "" H 1250 5500 50  0001 C CNN
+F 4 "823-22-034-10-000101" H 1250 5500 60  0001 C CNN "Mfg_Part_No"
+	1    1250 5500
+	1    0    0    -1
+$EndComp
+$Comp
+L Connector_Generic:Conn_02x17_Odd_Even P1
 U 1 1 5A4F0F21
-P 2550 5500
-F 0 "P1" H 2600 6400 50  0000 C CNN
-F 1 "Conn_02x17_Odd_Even" H 2600 4600 50  0000 C CNN
-F 2 "Sci-Bots:Pogo_Pin_Header_Straight_2x17_Pitch2.54mm" H 2550 5500 50  0001 C CNN
-F 3 "" H 2550 5500 50  0001 C CNN
-F 4 "823-22-034-10-000101" H 2550 5500 60  0001 C CNN "Mfg_Part_No"
-	1    2550 5500
-	1    0    0    -1
-$EndComp
-$Comp
-L CONN_02X17 P3
+P 2500 5500
+F 0 "P1" H 2550 6400 50  0000 C CNN
+F 1 "Conn_02x17_Odd_Even" H 2550 4600 50  0000 C CNN
+F 2 "Sci-Bots:Pogo_Pin_Header_Straight_2x17_Pitch2.54mm" H 2500 5500 50  0001 C CNN
+F 3 "" H 2500 5500 50  0001 C CNN
+F 4 "823-22-034-10-000101" H 2500 5500 60  0001 C CNN "Mfg_Part_No"
+	1    2500 5500
+	1    0    0    -1
+$EndComp
+$Comp
+L Connector_Generic:Conn_02x17_Odd_Even P3
 U 1 1 5A4F1091
-P 4050 5500
-F 0 "P3" H 4100 6400 50  0000 C CNN
-F 1 "Conn_02x17_Odd_Even" H 4100 4600 50  0000 C CNN
-F 2 "Sci-Bots:Pogo_Pin_Header_Straight_2x17_Pitch2.54mm" H 4050 5500 50  0001 C CNN
-F 3 "" H 4050 5500 50  0001 C CNN
-F 4 "823-22-034-10-000101" H 4050 5500 60  0001 C CNN "Mfg_Part_No"
-	1    4050 5500
-	1    0    0    -1
-$EndComp
-$Comp
-L CONN_02X17 P4
+P 4000 5500
+F 0 "P3" H 4050 6400 50  0000 C CNN
+F 1 "Conn_02x17_Odd_Even" H 4050 4600 50  0000 C CNN
+F 2 "Sci-Bots:Pogo_Pin_Header_Straight_2x17_Pitch2.54mm" H 4000 5500 50  0001 C CNN
+F 3 "" H 4000 5500 50  0001 C CNN
+F 4 "823-22-034-10-000101" H 4000 5500 60  0001 C CNN "Mfg_Part_No"
+	1    4000 5500
+	1    0    0    -1
+$EndComp
+$Comp
+L Connector_Generic:Conn_02x17_Odd_Even P4
 U 1 1 5A4F112A
-P 5350 5500
-F 0 "P4" H 5400 6400 50  0000 C CNN
-F 1 "Conn_02x17_Odd_Even" H 5400 4600 50  0000 C CNN
-F 2 "Sci-Bots:Pogo_Pin_Header_Straight_2x17_Pitch2.54mm" H 5350 5500 50  0001 C CNN
-F 3 "" H 5350 5500 50  0001 C CNN
-F 4 "823-22-034-10-000101" H 5350 5500 60  0001 C CNN "Mfg_Part_No"
-	1    5350 5500
-	1    0    0    -1
-$EndComp
-$Comp
-L CONN_02X25 J5
+P 5300 5500
+F 0 "P4" H 5350 6400 50  0000 C CNN
+F 1 "Conn_02x17_Odd_Even" H 5350 4600 50  0000 C CNN
+F 2 "Sci-Bots:Pogo_Pin_Header_Straight_2x17_Pitch2.54mm" H 5300 5500 50  0001 C CNN
+F 3 "" H 5300 5500 50  0001 C CNN
+F 4 "823-22-034-10-000101" H 5300 5500 60  0001 C CNN "Mfg_Part_No"
+	1    5300 5500
+	1    0    0    -1
+$EndComp
+$Comp
+L Connector_Generic:Conn_02x25_Odd_Even J5
 U 1 1 58C16B88
-P 6900 2200
-F 0 "J5" H 6900 3500 50  0000 C CNN
-F 1 "SFM-125-02-L-D-A" V 6900 1950 50  0000 C CNN
-F 2 "Sci-Bots:SFM-125-02-XXX-D-A" H 6900 1450 50  0001 C CNN
-F 3 "" H 6900 1450 50  0000 C CNN
-F 4 "SFM-125-02-L-D-A" H 6900 2200 60  0001 C CNN "Mfg_Part_No"
-	1    6900 2200
-	-1   0    0    1
-$EndComp
-$Comp
-L CONN_02X20 J6
+P 6950 2200
+F 0 "J5" H 6950 3500 50  0000 C CNN
+F 1 "SFM-125-02-L-D-A" V 7000 2200 50  0000 C CNN
+F 2 "Sci-Bots:SFM-125-02-XXX-D-A" H 6950 1450 50  0001 C CNN
+F 3 "" H 6950 1450 50  0000 C CNN
+F 4 "SFM-125-02-L-D-A" H 6950 2200 60  0001 C CNN "Mfg_Part_No"
+	1    6950 2200
+	-1   0    0    1
+$EndComp
+$Comp
+L Connector_Generic:Conn_02x20_Odd_Even J6
 U 1 1 58C168F5
-P 8250 1950
-F 0 "J6" H 8250 3000 50  0000 C CNN
-F 1 "SFM-120-02-L-D-A" V 8250 1950 50  0000 C CNN
-F 2 "Sci-Bots:SFM-120-02-XXX-D-A" H 8250 1000 50  0001 C CNN
-F 3 "" H 8250 1000 50  0000 C CNN
-F 4 "SFM-120-02-L-D-A" H 8250 1950 60  0001 C CNN "Mfg_Part_No"
-	1    8250 1950
-	-1   0    0    1
-$EndComp
-$Comp
-L CONN_02X20 J4
+P 8300 2000
+F 0 "J6" H 8300 3050 50  0000 C CNN
+F 1 "SFM-120-02-L-D-A" V 8350 2000 50  0000 C CNN
+F 2 "Sci-Bots:SFM-120-02-XXX-D-A" H 8300 1050 50  0001 C CNN
+F 3 "" H 8300 1050 50  0000 C CNN
+F 4 "SFM-120-02-L-D-A" H 8300 2000 60  0001 C CNN "Mfg_Part_No"
+	1    8300 2000
+	-1   0    0    1
+$EndComp
+$Comp
+L Connector_Generic:Conn_02x20_Odd_Even J4
 U 1 1 58C16354
-P 5600 1950
-F 0 "J4" H 5600 3000 50  0000 C CNN
-F 1 "SFM-120-02-L-D-A" V 5600 1950 50  0000 C CNN
-F 2 "Sci-Bots:SFM-120-02-XXX-D-A" H 5600 1000 50  0001 C CNN
-F 3 "" H 5600 1000 50  0000 C CNN
-F 4 "SFM-120-02-L-D-A" H 5600 1950 60  0001 C CNN "Mfg_Part_No"
-	1    5600 1950
+P 5650 2000
+F 0 "J4" H 5650 3050 50  0000 C CNN
+F 1 "SFM-120-02-L-D-A" V 5700 2000 50  0000 C CNN
+F 2 "Sci-Bots:SFM-120-02-XXX-D-A" H 5650 1050 50  0001 C CNN
+F 3 "" H 5650 1050 50  0000 C CNN
+F 4 "SFM-120-02-L-D-A" H 5650 2000 60  0001 C CNN "Mfg_Part_No"
+	1    5650 2000
 	-1   0    0    1
 $EndComp
@@
 Wire Wire Line
 	2400 1350 2500 1350
+Wire Wire Line
+	1150 1150 1150 1350
+Wire Wire Line
+	2500 1150 2500 1350
 $EndSCHEMATC

Commit message: Remove unnecessary vias and pass ERC
Parts:
- FB1, FB2: symbol Device:Ferrite_Bead_Small -> sci-bots:FERRITE
Connections:
- wire segments 28 -> 29
Other:
- note added: "PWR_FLAGS (to prevent ERC errors)"
- moved on the sheet: R1

Commit message: Fix BOM
Parts:
- C1, C2: MPN (none) -> CL21B104KBCNNNC; Manufacturer (none) -> Samsung; Mfg_Part_No CL21B104KBCNNNC -> (none)
- FB1, FB2: MPN (none) -> 742792040; Manufacturer (none) -> Würth Elektronik; Mfg_Part_No 742792040 -> (none)
- J4, J6: MPN (none) -> SFM-120-02-L-D-A; Manufacturer (none) -> Samtec; Mfg_Part_No SFM-120-02-L-D-A -> (none)
- J5: MPN (none) -> SFM-125-02-L-D-A; Manufacturer (none) -> Samtec; Mfg_Part_No SFM-125-02-L-D-A -> (none)
- P1, P2, P3, P4: MPN (none) -> 823-22-034-10-000101; Manufacturer (none) -> Mill-Max; Mfg_Part_No 823-22-034-10-000101 -> (none)
- P5, P6, P7, P8: MPN (none) -> DNP; Manufacturer (none) -> DNP
- R1: MPN (none) -> RC0805FR-0710KL; Manufacturer (none) -> Yageo; Mfg_Part_No RC0805FR-0710KL -> (none)
- U1: MPN (none) -> CAT24C02TDI-GT3A; Manufacturer (none) -> onsemi; Mfg_Part_No CAT24C02TDI-GT3A -> (none)
